File: boards/led/led.kicad_pcb (KiCad board)
At the start: 2 copper layers, 50 x 50 mm, 12 parts

Commit message: production: adopt pcb-kit's release flow (pcbkit.toml), v2.0 silkscreen labels
- pcbkit.toml: boards/*, JLC files only; pcbkit release --dry-run passes both boards (would release v2.0)
- silkscreen "v2" -> "v2.0" so pcbkit release re-stamps it; LED label moved to r = 12.2 mm to clear H3
- PRODUCTION.md: release/order steps, never-checked SOT-89/SOT-353 rotations, J1/J2 back BOM, overview
- LAYOUT/README/DESIGN: cleanup --dry-run result, release commands

Co-Authored-By: Claude Opus 5.5 <noreply@anthropic.com>
Other:
- board text added: "RGB LED v2.0"
- board text removed: "RGB LED v2"
Changed lines of the file:
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@@
 		)
 	)
-	(gr_text "RGB LED v2"
-		(at 150 113.4 90)
+	(gr_text "RGB LED v2.0"
+		(at 150 112.2 90)
 		(layer "F.SilkS")
 		(effects
